File: PCBs/troi/separation.brd (EAGLE design)
At the start: 100 x 80 mm, 14 parts, among them IC1 L7805ACV, Q1 IRLZ24NPBF

Commit message: Troi Value Changes
Just changed the value of the resistors in the potentiometer (potential divider).
Parts:
- R2: value 220k -> 2.2k
- R3: value 120k -> 1.2k
Changed lines of the file:
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@@
 <attribute name="VALUE" x="55.5244" y="47.7774" size="0.9906" layer="27" ratio="10"/>
 </element>
-<element name="R2" library="rcl" library_urn="urn:adsk.eagle:library:334" package="0204/7" package3d_urn="urn:adsk.eagle:package:23498/2" value="220k " x="30.48" y="57.15" smashed="yes">
+<element name="R2" library="rcl" library_urn="urn:adsk.eagle:library:334" package="0204/7" package3d_urn="urn:adsk.eagle:package:23498/2" value="2.2k" x="30.48" y="57.15" smashed="yes">
 <attribute name="NAME" x="27.94" y="58.4454" size="0.9906" layer="25" ratio="10"/>
 <attribute name="POPULARITY" value="79" x="48.26" y="13.97" size="1.778" layer="27" display="off"/>
@@
 <attribute name="VALUE" x="28.8544" y="56.6674" size="0.9906" layer="27" ratio="10"/>
 </element>
-<element name="R3" library="rcl" library_urn="urn:adsk.eagle:library:334" package="0204/7" package3d_urn="urn:adsk.eagle:package:23498/2" value="120k" x="57.15" y="57.15" smashed="yes">
+<element name="R3" library="rcl" library_urn="urn:adsk.eagle:library:334" package="0204/7" package3d_urn="urn:adsk.eagle:package:23498/2" value="1.2k" x="57.15" y="57.15" smashed="yes">
 <attribute name="NAME" x="54.61" y="58.4454" size="0.9906" layer="25" ratio="10"/>
 <attribute name="POPULARITY" value="79" x="85.09" y="13.97" size="1.778" layer="27" display="off"/>

Commit message: separation board arrangement
Parts:
- moved Q1 41.3 mm to (7.62, 39.4)
- moved IC1 33.6 mm to (7.62, 54.6)
- moved MCU-R 30.9 mm to (49.5, 73.7), turned to 180 degrees
- moved BATTERY_TERMINAL 30.5 mm to (7.62, 6.35)
- moved MCU-L 20.4 mm to (49.5, 67.3), turned to 180 degrees
- moved SERVO_PINS 14.5 mm to (26.7, 25.4)
- moved JP1 13.5 mm to (85.1, 58.4), turned to 90 degrees
